File: KiCad Proj/dumper/dumper.sch (KiCad schematic (older format))
At the start: 2 parts, among them J2 LINK PORT

Commit message: Finalized schematic and PCB
Parts:
- J2: value LINK PORT -> SPI
Changed lines of the file:
@@
 P 6350 4800
 F 0 "J2" H 6400 5117 50  0000 C CNN
-F 1 "LINK PORT" H 6400 5026 50  0000 C CNN
+F 1 "SPI" H 6400 5026 50  0000 C CNN
 F 2 "Connector_PinHeader_2.54mm:PinHeader_2x03_P2.54mm_Vertical" H 6350 4800 50  0001 C CNN
 F 3 "~" H 6350 4800 50  0001 C CNN
@@
 $EndComp
 $Sheet
-S 2600 2150 700  650
-U 61287E9C
-F0 "Cart Detection" 50
-F1 "voltage_switcher.sch" 50
-F2 "CART_VCC" I R 3300 2400 50
-F3 "GB_CART_H" I R 3300 2550 50
-$EndSheet
-$Sheet
-S 3850 3100 1900 2250
-U 611C0BE1
-F0 "Controller" 50
-F1 "controller.sch" 50
-F2 "CART_CS" O R 5750 4050 50
-F3 "SWITCH_TRANSCEIVER" O R 5750 3250 50
-F4 "SS" O R 5750 4800 50
-F5 "MOSI" O R 5750 4700 50
-F6 "MISO" O R 5750 4600 50
-F7 "SCK" O R 5750 4900 50
-F8 "ADDRESS_DATA" O R 5750 3350 50
-F9 "ADDRESS_CLK" O R 5750 3450 50
-F10 "ADDRESS_LATCH" O R 5750 3550 50
-F11 "CART_RD" O R 5750 4150 50
-F12 "CART_WR" O R 5750 4250 50
-F13 "SCL" O R 5750 5150 50
-F14 "SDA" O R 5750 5250 50
-F15 "D[0..7]" B R 5750 3150 50
-F16 "GB_CART_H" O L 3850 3150 50
-$EndSheet
-$Sheet
 S 8500 3100 900  650
 U 61279BC9
@@
 Wire Bus Line
 	8150 3350 8500 3350
+$Sheet
+S 3850 3100 1900 2250
+U 611C0BE1
+F0 "Controller" 50
+F1 "controller.sch" 50
+F2 "CART_CS" O R 5750 4050 50
+F3 "SWITCH_TRANSCEIVER" O R 5750 3250 50
+F4 "SS" O R 5750 4800 50
+F5 "MOSI" O R 5750 4700 50
+F6 "MISO" O R 5750 4600 50
+F7 "SCK" O R 5750 4900 50
+F8 "ADDRESS_DATA" O R 5750 3350 50
+F9 "ADDRESS_CLK" O R 5750 3450 50
+F10 "ADDRESS_LATCH" O R 5750 3550 50
+F11 "CART_RD" O R 5750 4150 50
+F12 "CART_WR" O R 5750 4250 50
+F13 "SCL" O R 5750 5150 50
+F14 "SDA" O R 5750 5250 50
+F15 "D[0..7]" B R 5750 3150 50
+F16 "GB_CART_H" O L 3850 3150 50
+$EndSheet
+$Sheet
+S 2600 2150 700  650
+U 61287E9C
+F0 "Cart Detection" 50
+F1 "voltage_switcher.sch" 50
+F2 "CART_VCC" I R 3300 2400 50
+F3 "GB_CART_H" I R 3300 2550 50
+$EndSheet
 $EndSCHEMATC
