File: KiCad Proj/dumper/memory_block_data.sch (KiCad schematic (older format))
At the start: 6 parts, among them U1 74HC595, U2 SN74LVC8T245PWR, U3 74HC595, U4 SN74LVC8T245PWR, U5 SN74LVC8T245PWR

Commit message: Finalized schematic and PCB
Connections:
- net +3V3: now also U2.23 (VccB), U2.24 (VccB), U4.23 (VccB), U4.24 (VccB), U5.23 (VccB), U5.24 (VccB); no longer U1.16 (VCC), U2.1 (VccA), U2.2 (DIR), U3.16 (VCC), U4.1 (VccA), U4.2 (DIR), U5.1 (VccA)
- net +5V: now also U1.16 (VCC), U2.1 (VccA), U2.2 (DIR), U3.16 (VCC), U4.1 (VccA), U4.2 (DIR), U5.1 (VccA); no longer U2.23 (VccB), U2.24 (VccB), U4.23 (VccB), U4.24 (VccB), U5.23 (VccB), U5.24 (VccB)
- net A0: now also U2.21 (B1); no longer U2.14 (B8)
- net A1: now also U2.20 (B2); no longer U2.15 (B7)
- net A10: now also U4.19 (B3); no longer U4.16 (B6)
- net A11: now also U4.18 (B4); no longer U4.17 (B5)
- net A12: now also U4.17 (B5); no longer U4.18 (B4)
- net A13: now also U4.16 (B6); no longer U4.19 (B3)
- net A14: now also U4.15 (B7); no longer U4.20 (B2)
- net A15: now also U4.14 (B8); no longer U4.21 (B1)
- net A2: now also U2.19 (B3); no longer U2.16 (B6)
- net A3: now also U2.18 (B4); no longer U2.17 (B5)
- net A4: now also U2.17 (B5); no longer U2.18 (B4)
- net A5: now also U2.16 (B6); no longer U2.19 (B3)
- net A6: now also U2.15 (B7); no longer U2.20 (B2)
- net A7: now also U2.14 (B8); no longer U2.21 (B1)
- net A8: now also U4.21 (B1); no longer U4.14 (B8)
- net A9: now also U4.20 (B2); no longer U4.15 (B7)
- net ADDRESS_DATA: now also U3.14 (SER); no longer U1.14 (SER)
- net GND: now also U1.8 (GND), U1.9 (QH'), U3.8 (GND); no longer U2.22 (OE)
- net QA_B: now reaches U2.10 (A8)
- net QA_B: now also U1.15 (QA); no longer U1.7 (QH)
- net QH_B: now reaches U2.3 (A1)
- net QH_B: now also U1.7 (QH); no longer U1.15 (QA)
- net QB_B: now reaches U1.1 (QB)
- net QB_B: now also U2.9 (A7); no longer U2.4 (A2)
- net QC_B: now reaches U1.2 (QC)
- net QC_B: now also U2.8 (A6); no longer U2.5 (A3)
- net QD_B: now reaches U1.3 (QD)
- net QD_B: now also U2.7 (A5); no longer U2.6 (A4)
- net QE_B: now reaches U1.4 (QE)
- net QE_B: now also U2.6 (A4); no longer U2.7 (A5)
- net QF_B: now reaches U1.5 (QF)
- net QF_B: now also U2.5 (A3); no longer U2.8 (A6)
- net QG_B: now reaches U1.6 (QG)
- net QG_B: now also U2.4 (A2); no longer U2.9 (A7)
- net QA_A: now reaches U4.10 (A8)
- net QA_A: now also U3.15 (QA); no longer U3.7 (QH)
- net QH_A: now reaches U4.3 (A1)
- net QH_A: now also U3.7 (QH); no longer U3.15 (QA)
- net QB_A: now reaches U3.1 (QB)
- net QB_A: now also U4.9 (A7); no longer U4.4 (A2)
- net QC_A: now reaches U3.2 (QC)
- net QC_A: now also U4.8 (A6); no longer U4.5 (A3)
- net QD_A: now reaches U3.3 (QD)
- net QD_A: now also U4.7 (A5); no longer U4.6 (A4)
- net QE_A: now reaches U3.4 (QE)
- net QE_A: now also U4.6 (A4); no longer U4.7 (A5)
- net QF_A: now reaches U3.5 (QF)
- net QF_A: now also U4.5 (A3); no longer U4.8 (A6)
- net QG_A: now reaches U3.6 (QG)
- net QG_A: now also U4.4 (A2); no longer U4.9 (A7)
- net at U3.9 (QH'): now also U1.14 (SER)
Other:
- moved on the sheet: R4, U1, U2, U3, U4
