File: KiCad Proj/KiCad Proj/dumper/cart_slot.sch (KiCad schematic (older format))
At the start: 5 parts, among them J1 CartBus

Commit message: Fixed up the schematic and PCB for two very severe omissions
I forgot to translate the WR, RD, and CS pins and added a transceiver for those

I also forgot that the transceivers should have CART_VCC on VccB
Connections:
- net CART_CS renamed TRANS_CART_CS
- net CART_WR renamed TRANS_CART_WR
Changed lines of the file:
@@
 $Descr A4 11693 8268
 encoding utf-8
-Sheet 4 5
+Sheet 2 5
 Title "Italian Retro Guy's Cart Dumper - Cartridge Slot"
 Date ""
@@
 CART_VCC
 Text HLabel 4400 5050 0    50   Input ~ 0
-CART_CS
+TRANS_CART_CS
 Text HLabel 4400 5150 0    50   Input ~ 0
-CART_RD
+TRANS_CART_RD
 Text HLabel 4400 5250 0    50   Input ~ 0
-CART_WR
+TRANS_CART_WR
 $Comp
 L Device:R R?
@@
 Text Label 6050 3350 2    50   ~ 0
 TD0
-Text Label 5800 2950 2    50   ~ 0
-TD[0..7]
+Text Label 5800 4250 2    50   ~ 0
+A[0..15]
 Wire Wire Line
 	4400 5050 5050 5050
